File: kicad/mr107_802.3af/mr107.kicad_pcb (KiCad board)
At the start: 2 copper layers, 35.8 x 70.1 mm, 64 parts, among them J1 USBA DS1095B-R, J2 gnd, J3 mosi, J4 miso, J5 sclk, J6 reset, J7 gnd, J8 gnd, J9 PW, T1 HY931147C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

Commit message: удалено:       kicad/mr107_802.3af/gerber/Border.gbr 	удалено:       kicad/mr107_802.3af/gerber/Bottom.gbr 	удалено:       kicad/mr107_802.3af/gerber/MaskBottom.gbr 	удалено:       kicad/mr107_802.3af/gerber/MaskTop.gbr 	удалено:       kicad/mr107_802.3af/gerber/NCData.drl 	удалено:       kicad/mr107_802.3af/gerber/Top.gbr 	изменено:      kicad/mr107_802.3af/gerber/mk-gerber.sh 	удалено:       kicad/mr107_802.3af/gerber/mk-gerber.sh~ 	удалено:       kicad/mr107_802.3af/gerber/mr107-job.gbrjob 	изменено:      kicad/mr107_802.3af/gerber/mr107.zip 	удалено:       kicad/mr107_802.3af/mr107-backups/mr107-2023-12-18_145009.zip 	удалено:       kicad/mr107_802.3af/mr107-backups/mr107-2023-12-18_150211.zip 	удалено:       kicad/mr107_802.3af/mr107-backups/mr107-2023-12-18_150828.zip 	удалено:       kicad/mr107_802.3af/mr107-backups/mr107-2023-12-18_153503.zip 	изменено:      kicad/mr107_802.3af/mr107.kicad_pcb 	изменено:      kicad/mr107_802.3af/mr107.kicad_prl
Parts:
- moved R9 1.93 mm to (78.3, 116.0)
Routing:
- net act: track 3.24 -> 5.18 mm
- net Net-(R9-Pad1): track 45.8 -> 43.9 mm
Changed lines of the file:
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@@
   )
   (footprint "Resistor_SMD:R_0603_1608Metric" (layer "F.Cu")
-    (at 80.2 115.98 -90)
+    (at 78.27 115.99 -90)
     (descr "Resistor SMD 0603 (1608 Metric), square (rectangular) end terminal, IPC_7351 nominal, (Body size source: IPC-SM-782 page 72, https://www.pcb-3d.com/wordpress/wp-content/uploads/ipc-sm-782a_amendment_1_and_2.pdf), generated with kicad-footprint-generator")
     (tags "resistor")
@@
   (segment (start 78.652893 63.992107) (end 79.71 62.935) (width 0.25) (layer "B.Cu") (net 78))
   (arc (start 78.36 64.699214) (mid 78.43612 64.316531) (end 78.652893 63.992107) (width 0.25) (layer "B.Cu") (net 78))
+  (segment (start 69.78 85.714214) (end 69.78 108.095786) (width 0.25) (layer "F.Cu") (net 79))
   (segment (start 75.17 81.29) (end 75.17 81.325786) (width 0.25) (layer "F.Cu") (net 79))
-  (segment (start 69.78 85.714214) (end 69.78 108.095786) (width 0.25) (layer "F.Cu") (net 79))
+  (segment (start 70.072893 108.802893) (end 75.027107 113.757107) (width 0.25) (layer "F.Cu") (net 79))
+  (segment (start 73.995786 82.5) (end 72.994214 82.5) (width 0.25) (layer "F.Cu") (net 79))
+  (segment (start 74.877107 82.032893) (end 74.702893 82.207107) (width 0.25) (layer "F.Cu") (net 79))
+  (segment (start 75.734214 114.05) (end 76.740786 114.05) (width 0.25) (layer "F.Cu") (net 79))
+  (segment (start 77.447893 114.342893) (end 78.27 115.165) (width 0.25) (layer "F.Cu") (net 79))
   (segment (start 72.287107 82.792893) (end 70.072893 85.007107) (width 0.25) (layer "F.Cu") (net 79))
-  (segment (start 75.734214 114.05) (end 78.680786 114.05) (width 0.25) (layer "F.Cu") (net 79))
-  (segment (start 73.995786 82.5) (end 72.994214 82.5) (width 0.25) (layer "F.Cu") (net 79))
-  (segment (start 70.072893 108.802893) (end 75.027107 113.757107) (width 0.25) (layer "F.Cu") (net 79))
-  (segment (start 74.877107 82.032893) (end 74.702893 82.207107) (width 0.25) (layer "F.Cu") (net 79))
-  (segment (start 79.387893 114.342893) (end 80.2 115.155) (width 0.25) (layer "F.Cu") (net 79))
   (via (at 75.17 81.29) (size 0.8) (drill 0.4) (layers "F.Cu" "B.Cu") (net 79))
+  (arc (start 69.78 108.095786) (mid 69.85612 108.478469) (end 70.072893 108.802893) (width 0.25) (layer "F.Cu") (net 79))
+  (arc (start 77.447893 114.342893) (mid 77.12347 114.12612) (end 76.740786 114.05) (width 0.25) (layer "F.Cu") (net 79))
+  (arc (start 75.17 81.325786) (mid 75.09388 81.70847) (end 74.877107 82.032893) (width 0.25) (layer "F.Cu") (net 79))
+  (arc (start 72.994214 82.5) (mid 72.611531 82.57612) (end 72.287107 82.792893) (width 0.25) (layer "F.Cu") (net 79))
+  (arc (start 75.027107 113.757107) (mid 75.351531 113.97388) (end 75.734214 114.05) (width 0.25) (layer "F.Cu") (net 79))
   (arc (start 70.072893 85.007107) (mid 69.85612 85.331531) (end 69.78 85.714214) (width 0.25) (layer "F.Cu") (net 79))
-  (arc (start 75.734214 114.05) (mid 75.351531 113.97388) (end 75.027107 113.757107) (width 0.25) (layer "F.Cu") (net 79))
-  (arc (start 72.994214 82.5) (mid 72.611531 82.57612) (end 72.287107 82.792893) (width 0.25) (layer "F.Cu") (net 79))
-  (arc (start 75.17 81.325786) (mid 75.09388 81.70847) (end 74.877107 82.032893) (width 0.25) (layer "F.Cu") (net 79))
-  (arc (start 69.78 108.095786) (mid 69.85612 108.478469) (end 70.072893 108.802893) (width 0.25) (layer "F.Cu") (net 79))
   (arc (start 74.702893 82.207107) (mid 74.37847 82.42388) (end 73.995786 82.5) (width 0.25) (layer "F.Cu") (net 79))
-  (arc (start 79.387893 114.342893) (mid 79.06347 114.12612) (end 78.680786 114.05) (width 0.25) (layer "F.Cu") (net 79))
   (segment (start 76.012893 81.56) (end 75.647107 81.56) (width 0.25) (layer "B.Cu") (net 79))
   (segment (start 76.408553 81.748553) (end 76.366446 81.706446) (width 0.25) (layer "B.Cu") (net 79))
@@
   (arc (start 75.877893 117.657107) (mid 75.55347 117.87388) (end 75.170786 117.95) (width 0.25) (layer "F.Cu") (net 91))
   (arc (start 72.337107 118.242893) (mid 72.66153 118.02612) (end 73.044214 117.95) (width 0.25) (layer "F.Cu") (net 91))
-  (segment (start 80.492893 117.982893) (end 81.9 119.39) (width 0.25) (layer "F.Cu") (net 92))
-  (segment (start 80.2 116.805) (end 80.2 117.275786) (width 0.25) (layer "F.Cu") (net 92))
-  (arc (start 80.492893 117.982893) (mid 80.27612 117.65847) (end 80.2 117.275786) (width 0.25) (layer "F.Cu") (net 92))
+  (segment (start 79.567107 119.097107) (end 78.562893 118.092893) (width 0.25) (layer "F.Cu") (net 92))
+  (segment (start 81.9 119.39) (end 80.274214 119.39) (width 0.25) (layer "F.Cu") (net 92))
+  (segment (start 78.27 117.385786) (end 78.27 116.815) (width 0.25) (layer "F.Cu") (net 92))
+  (arc (start 78.562893 118.092893) (mid 78.34612 117.76847) (end 78.27 117.385786) (width 0.25) (layer "F.Cu") (net 92))
+  (arc (start 79.567107 119.097107) (mid 79.89153 119.31388) (end 80.274214 119.39) (width 0.25) (layer "F.Cu") (net 92))
   (segment (start 61.23 117.51) (end 59.802893 116.082893) (width 0.25) (layer "F.Cu") (net 93))
   (segment (start 59.51 115.375786) (end 59.51 114.564214) (width 0.25) (layer "F.Cu") (net 93))
