File: kicad/mr107/mr107.kicad_sch (KiCad schematic)
At the start: 72 parts, among them J1 USBA DS1095B-R, J10 L-KLS12, J2 RxD, J3 mosi, J4 miso, J5 sclk, J6 reset, J7 gnd, J8 TxD, J9 PW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

Commit message: удалено:       kicad/mr107/mr107-backups/mr107-2023-12-12_103509.zip 	удалено:       kicad/mr107/mr107-backups/mr107-2023-12-12_104452.zip 	удалено:       kicad/mr107/mr107-backups/mr107-2023-12-12_105008.zip 	удалено:       kicad/mr107/mr107-backups/mr107-2023-12-12_105739.zip 	изменено:      kicad/mr107/mr107.kicad_pcb 	изменено:      kicad/mr107/mr107.kicad_sch
Parts:
- removed Y3: 8MHz, Crystal:Resonator_SMD_Murata_CSTxExxV-3Pin_3.0x1.1mm, symbol Device:Crystal_GND2
- added R17: 1M, Resistor_SMD:R_0402_1005Metric, symbol Device:R
- added Y3: 8MHz, Crystal:Resonator_SMD_Murata_CSTxExxV-3Pin_3.0x1.1mm, symbol Device:Crystal_GND2_Small
- gave numbers to parts that had none: 2
Connections:
- net GND: now also Y3.2
- net at U2.8 (XTAL2/PB7): now also R17.2, Y3.1
- net at U2.7 (XTAL1/PB6): now also R17.1, Y3.3
Changed lines of the file:
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@@
   (junction (at 149.86 170.815) (diameter 0) (color 0 0 0 0)
   )
+  (junction (at 64.77 52.07) (diameter 0) (color 0 0 0 0)
+  )
   (junction (at 142.24 33.655) (diameter 0) (color 0 0 0 0)
   )
@@
   )
   (junction (at 116.205 26.035) (diameter 0) (color 0 0 0 0)
+  )
+  (junction (at 72.39 54.61) (diameter 0) (color 0 0 0 0)
   )
   (junction (at 50.165 155.575) (diameter 0) (color 0 0 0 0)
@@
     (stroke (width 0) (type default) (color 0 0 0 0))
   )
+  (wire (pts (xy 64.77 52.07) (xy 78.74 52.07))
+    (stroke (width 0) (type default) (color 0 0 0 0))
+  )
   (wire (pts (xy 108.585 142.875) (xy 97.79 142.875))
     (stroke (width 0) (type default) (color 0 0 0 0))
@@
     (stroke (width 0) (type default) (color 0 0 0 0))
   )
-  (wire (pts (xy 72.39 52.07) (xy 72.39 55.245))
-    (stroke (width 0) (type default) (color 0 0 0 0))
-  )
   (wire (pts (xy 76.835 117.475) (xy 81.915 117.475))
     (stroke (width 0) (type default) (color 0 0 0 0))
@@
     (stroke (width 0) (type default) (color 0 0 0 0))
   )
-  (wire (pts (xy 64.77 54.61) (xy 64.77 55.245))
-    (stroke (width 0) (type default) (color 0 0 0 0))
-  )
   (wire (pts (xy 121.92 55.88) (xy 125.73 55.88))
     (stroke (width 0) (type default) (color 0 0 0 0))
@@
     (stroke (width 0) (type default) (color 0 0 0 0))
   )
+  (wire (pts (xy 72.39 54.61) (xy 72.39 57.15))
+    (stroke (width 0) (type default) (color 0 0 0 0))
+  )
+  (wire (pts (xy 72.39 54.61) (xy 73.66 54.61))
+    (stroke (width 0) (type default) (color 0 0 0 0))
+  )
   (wire (pts (xy 144.145 125.095) (xy 144.145 126.365))
     (stroke (width 0) (type default) (color 0 0 0 0))
@@
     (stroke (width 0) (type default) (color 0 0 0 0))
   )
+  (wire (pts (xy 78.74 52.07) (xy 78.74 54.61))
+    (stroke (width 0) (type default) (color 0 0 0 0))
+  )
   (wire (pts (xy 42.545 168.91) (xy 42.545 179.07))
     (stroke (width 0) (type default) (color 0 0 0 0))
@@
     (stroke (width 0) (type default) (color 0 0 0 0))
   )
-  (wire (pts (xy 62.865 54.61) (xy 64.77 54.61))
+  (wire (pts (xy 62.865 54.61) (xy 72.39 54.61))
     (stroke (width 0) (type default) (color 0 0 0 0))
   )
@@
     (stroke (width 0) (type default) (color 0 0 0 0))
   )
-  (wire (pts (xy 62.865 52.07) (xy 72.39 52.07))
+  (wire (pts (xy 62.865 52.07) (xy 64.77 52.07))
     (stroke (width 0) (type default) (color 0 0 0 0))
   )
@@
   )
   (wire (pts (xy 34.925 165.735) (xy 34.925 171.45))
+    (stroke (width 0) (type default) (color 0 0 0 0))
+  )
+  (wire (pts (xy 64.77 52.07) (xy 64.77 57.15))
     (stroke (width 0) (type default) (color 0 0 0 0))
   )
@@
     (pin "2")
   )
-  (symbol (lib_id "power:GND") (at 68.58 60.325 0) (unit 1)
-    (in_bom yes) (on_board yes) (fields_autoplaced)
-    (property "Reference" "#PWR0115" (id 0) (at 68.58 66.675 0)
-      (effects (font (size 1.27 1.27)) hide)
-    )
-    (property "Value" "GND" (id 1) (at 68.58 64.7684 0)
-      (effects (font (size 1.27 1.27)) hide)
-    )
-    (property "Footprint" "" (id 2) (at 68.58 60.325 0)
-      (effects (font (size 1.27 1.27)) hide)
-    )
-    (property "Datasheet" "" (id 3) (at 68.58 60.325 0)
+  (symbol (lib_id "power:GND") (at 76.2 57.15 0) (unit 1)
+    (in_bom yes) (on_board yes) (fields_autoplaced)
+    (property "Reference" "#PWR0115" (id 0) (at 76.2 63.5 0)
+      (effects (font (size 1.27 1.27)) hide)
+    )
+    (property "Value" "GND" (id 1) (at 76.2 61.5934 0)
+      (effects (font (size 1.27 1.27)) hide)
+    )
+    (property "Footprint" "" (id 2) (at 76.2 57.15 0)
+      (effects (font (size 1.27 1.27)) hide)
+    )
+    (property "Datasheet" "" (id 3) (at 76.2 57.15 0)
       (effects (font (size 1.27 1.27)) hide)
     )
@@
     (pin "2")
   )
-  (symbol (lib_id "Device:Crystal_GND2") (at 68.58 55.245 0) (unit 1)
-    (in_bom yes) (on_board yes)
-    (property "Reference" "Y3" (id 0) (at 75.565 54.61 0))
-    (property "Value" "8MHz" (id 1) (at 75.565 56.515 0))
-    (property "Footprint" "Crystal:Resonator_SMD_Murata_CSTxExxV-3Pin_3.0x1.1mm" (id 2) (at 68.58 55.245 0)
-      (effects (font (size 1.27 1.27)) hide)
-    )
-    (property "Datasheet" "~" (id 3) (at 68.58 55.245 0)
-      (effects (font (size 1.27 1.27)) hide)
-    )
-    (pin "1")
-    (pin "2")
-    (pin "3")
-  )
   (symbol (lib_id "Device:Crystal_GND24_Small") (at 39.37 171.45 0) (unit 1)
     (in_bom yes) (on_board yes)
@@
   (symbol (lib_id "My-Library:Conn") (at 73.025 69.85 0) (unit 1)
     (in_bom yes) (on_board yes)
-    (property "Reference" "J?" (id 0) (at 73.7362 69.0153 0)
+    (property "Reference" "J11" (id 0) (at 73.7362 69.0153 0)
       (effects (font (size 1.27 1.27)) (justify left) hide)
     )
@@
     (pin "9")
   )
+  (symbol (lib_id "Device:R") (at 68.58 57.15 90) (unit 1)
+    (in_bom yes) (on_board yes)
+    (property "Reference" "R17" (id 0) (at 68.58 59.69 90))
+    (property "Value" "1M" (id 1) (at 68.58 61.595 90))
+    (property "Footprint" "Resistor_SMD:R_0402_1005Metric" (id 2) (at 68.58 58.928 90)
+      (effects (font (size 1.27 1.27)) hide)
+    )
+    (property "Datasheet" "~" (id 3) (at 68.58 57.15 0)
+      (effects (font (size 1.27 1.27)) hide)
+    )
+    (pin "1")
+    (pin "2")
+  )
   (symbol (lib_id "My-Library:Conn") (at 66.675 26.035 180) (unit 1)
     (in_bom yes) (on_board yes)
@@
     (pin "1")
   )
+  (symbol (lib_id "Device:Crystal_GND2_Small") (at 76.2 54.61 0) (unit 1)
+    (in_bom yes) (on_board yes)
+    (property "Reference" "Y3" (id 0) (at 76.2 49.5132 0)
+      (effects (font (size 1.27 1.27)) hide)
+    )
+    (property "Value" "8MHz" (id 1) (at 81.915 53.34 0))
+    (property "Footprint" "Crystal:Resonator_SMD_Murata_CSTxExxV-3Pin_3.0x1.1mm" (id 2) (at 76.2 54.61 0)
+      (effects (font (size 1.27 1.27)) hide)
+    )
+    (property "Datasheet" "~" (id 3) (at 76.2 54.61 0)
+      (effects (font (size 1.27 1.27)) hide)
+    )
+    (pin "1")
+    (pin "2")
+    (pin "3")
+  )
   (symbol (lib_id "Device:C") (at 139.7 52.07 0) (unit 1)
     (in_bom yes) (on_board yes)
@@
   (symbol (lib_id "My-Library:Conn") (at 73.025 72.39 0) (unit 1)
     (in_bom yes) (on_board yes)
-    (property "Reference" "J?" (id 0) (at 73.7362 71.5553 0)
+    (property "Reference" "J12" (id 0) (at 73.7362 71.5553 0)
       (effects (font (size 1.27 1.27)) (justify left) hide)
     )
@@
     )
     (path "/62840a42-d90d-427c-ad9f-a984bc00595d"
-      (reference "J?") (unit 1) (value "mosi") (footprint "lib:conn_mini")
+      (reference "J11") (unit 1) (value "mosi") (footprint "lib:conn_mini")
     )
     (path "/b7efb4eb-5304-4752-b042-629f4172654c"
-      (reference "J?") (unit 1) (value "mosi") (footprint "lib:conn_mini")
+      (reference "J12") (unit 1) (value "mosi") (footprint "lib:conn_mini")
     )
     (path "/2be56d09-aac9-4f41-8d95-54c125ebb9b4"
@@
       (reference "R16") (unit 1) (value "75") (footprint "Resistor_SMD:R_0603_1608Metric")
     )
+    (path "/68af7bec-e982-4bb4-b691-4ee3716c342d"
+      (reference "R17") (unit 1) (value "1M") (footprint "Resistor_SMD:R_0402_1005Metric")
+    )
     (path "/08612cff-1192-476f-83ad-6ad1ebc12440"
       (reference "U1") (unit 1) (value "W5500") (footprint "Package_QFP:LQFP-48_7x7mm_P0.5mm")
@@
       (reference "Y2") (unit 1) (value "12MHz") (footprint "Crystal:Crystal_SMD_0603-4Pin_6.0x3.5mm")
     )
-    (path "/528196b2-5b8b-4392-9ebd-44b7e4d19b98"
+    (path "/adc1aba7-843a-43a3-af87-5110a8fe221d"
       (reference "Y3") (unit 1) (value "8MHz") (footprint "Crystal:Resonator_SMD_Murata_CSTxExxV-3Pin_3.0x1.1mm")
     )

Commit message: изменено:      kicad/mr107/gerber/mr107.zip 	изменено:      kicad/mr107/mr107.kicad_pcb 	изменено:      kicad/mr107/mr107.kicad_sch
Connections:
- net RST_ETH: now also U2.9 (PD5); no longer U2.25 (PC2)
Other:
- moved on the sheet: D2
Changed lines of the file:
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@@
   (no_connect (at 108.585 85.09))
   (no_connect (at 62.865 36.83))
-  (no_connect (at 62.865 92.71))
+  (no_connect (at 62.865 64.77))
   (no_connect (at 32.385 41.91))
   (no_connect (at 62.865 59.69))
@@
     (stroke (width 0) (type default) (color 0 0 0 0))
   )
+  (wire (pts (xy 62.865 92.71) (xy 63.5 92.71))
+    (stroke (width 0) (type default) (color 0 0 0 0))
+  )
   (wire (pts (xy 141.605 160.655) (xy 144.78 160.655))
     (stroke (width 0) (type default) (color 0 0 0 0))
@@
     (stroke (width 0) (type default) (color 0 0 0 0))
   )
-  (wire (pts (xy 72.39 90.17) (xy 74.93 90.17))
+  (wire (pts (xy 72.39 90.17) (xy 80.645 90.17))
     (stroke (width 0) (type default) (color 0 0 0 0))
   )
@@
   )
   (wire (pts (xy 46.99 142.875) (xy 50.165 142.875))
-    (stroke (width 0) (type default) (color 0 0 0 0))
-  )
-  (wire (pts (xy 62.865 64.77) (xy 65.405 64.77))
     (stroke (width 0) (type default) (color 0 0 0 0))
   )
@@
     )
   )
-  (global_label "RST_ETH" (shape input) (at 65.405 64.77 0) (fields_autoplaced)
+  (global_label "RST_ETH" (shape input) (at 63.5 92.71 0) (fields_autoplaced)
     (effects (font (size 1.27 1.27)) (justify left))
-    (property "Обозначения листов" "${INTERSHEET_REFS}" (id 0) (at 75.68 64.6906 0)
+    (property "Обозначения листов" "${INTERSHEET_REFS}" (id 0) (at 73.775 92.6306 0)
       (effects (font (size 1.27 1.27)) (justify left) hide)
     )
@@
     (pin "2")
   )
-  (symbol (lib_id "Device:LED") (at 74.93 93.98 90) (unit 1)
-    (in_bom yes) (on_board yes)
-    (property "Reference" "D2" (id 0) (at 78.105 93.98 90))
-    (property "Value" "LED" (id 1) (at 72.4971 95.5675 0)
-      (effects (font (size 1.27 1.27)) hide)
-    )
-    (property "Footprint" "LED_SMD:LED_0603_1608Metric" (id 2) (at 74.93 93.98 0)
-      (effects (font (size 1.27 1.27)) hide)
-    )
-    (property "Datasheet" "~" (id 3) (at 74.93 93.98 0)
+  (symbol (lib_id "Device:LED") (at 80.645 93.98 90) (unit 1)
+    (in_bom yes) (on_board yes)
+    (property "Reference" "D2" (id 0) (at 83.82 93.98 90))
+    (property "Value" "LED" (id 1) (at 78.2121 95.5675 0)
+      (effects (font (size 1.27 1.27)) hide)
+    )
+    (property "Footprint" "LED_SMD:LED_0603_1608Metric" (id 2) (at 80.645 93.98 0)
+      (effects (font (size 1.27 1.27)) hide)
+    )
+    (property "Datasheet" "~" (id 3) (at 80.645 93.98 0)
       (effects (font (size 1.27 1.27)) hide)
     )
@@
     (pin "2")
   )
-  (symbol (lib_id "power:GND") (at 74.93 97.79 0) (unit 1)
-    (in_bom yes) (on_board yes) (fields_autoplaced)
-    (property "Reference" "#PWR0102" (id 0) (at 74.93 104.14 0)
-      (effects (font (size 1.27 1.27)) hide)
-    )
-    (property "Value" "GND" (id 1) (at 74.93 102.2334 0)
-      (effects (font (size 1.27 1.27)) hide)
-    )
-    (property "Footprint" "" (id 2) (at 74.93 97.79 0)
-      (effects (font (size 1.27 1.27)) hide)
-    )
-    (property "Datasheet" "" (id 3) (at 74.93 97.79 0)
-      (effects (font (size 1.27 1.27)) hide)
-    )
+  (symbol (lib_id "power:GND") (at 80.645 97.79 0) (unit 1)
+    (in_bom yes) (on_board yes) (fields_autoplaced)
+    (property "Reference" "#PWR0102" (id 0) (at 80.645 104.14 0)
+      (effects (font (size 1.27 1.27)) hide)
+    )
+    (property "Value" "GND" (id 1) (at 80.645 102.2334 0)
+      (effects (font (size 1.27 1.27)) hide)
+    )
+    (property "Footprint" "" (id 2) (at 80.645 97.79 0)
+      (effects (font (size 1.27 1.27)) hide)
+    )
+    (property "Datasheet" "" (id 3) (at 80.645 97.79 0)
+      (effects (font (size 1.27 1.27)) hide)
+    )
